File: hardware/ptcontroller/ptcontroller.kicad_pcb (KiCad board)
At the start: 2 copper layers, 1 part

Commit message: saved pcb
Parts:
- removed REF**: TRIM_P0915N-FC15BR100K, P0915N-FC15BR100K:TRIM_P0915N-FC15BR100K
- added A1: Arduino_Mega2560_R3_Shield, PCM_arduino-library:Arduino_Mega2560_R3_Shield, F.Cu at (100.6, 129.5)
- added R1: P0915N-FC15BR100K, P0915N-FC15BR100K:TRIM_P0915N-FC15BR100K, F.Cu at (160.0, 17.8)
